Commit message: Collision model fix

File: jackal_kinova_gazebo/urdf/gen3_lite/6dof/urdf/gen3_lite_macro.xacro (robot description, xacro)
@@ -216,4 +216,10 @@
       </material>
     </visual>
+    <collision>
+      <origin xyz="-0.175 -0.01 -1.15" rpy="${PI/2} 0 ${PI/2}"/>
+      <geometry>
+        <mesh filename="package://jackal_kinova_gazebo/meshes/gen3_lite_camera_bracket.STL"/>
+      </geometry>
+    </collision>
   </link>
   <joint name="hand_camera_bracket_joint" type="fixed">

File: jackal_kinova_gazebo/urdf/include/d435.urdf.xacro (robot description, xacro)
@@ -45,10 +45,4 @@
         </geometry>
       </visual>
-      <collision>
-        <origin xyz="0 ${-d435_cam_depth_py} 0" rpy="0 0 0"/>
-        <geometry>
-          <box size="${d435_cam_depth} ${d435_cam_width} ${d435_cam_height}"/>
-        </geometry>
-      </collision>
       <inertial>
         <mass value="0.564" />

File: jackal_kinova_gazebo/urdf/include/tim571.urdf.xacro (robot description, xacro)
@@ -13,10 +13,4 @@
         <inertia ixx="${0.0833333 * mass * (width * width + height * height)}" ixy="0.0" ixz="0.0" iyy="${0.0833333 * mass * (length * length + height * height)}" iyz="0.0" izz="${0.0833333 * mass * (length * length + width * width)}" />
       </inertial>
-      <collision>
-        <origin xyz="0 0 -0.026" rpy="3.1415926 0 0"/>
-        <geometry>
-          <mesh filename="package://jackal_kinova_gazebo/meshes/include/tim571.stl"/>
-        </geometry>
-      </collision>
     </link>
     <joint name="${name}_joint" type="fixed">

File: jackal_kinova_gazebo/urdf/jackal_kinova.urdf.xacro (robot description, xacro)
@@ -6,4 +6,5 @@
   <xacro:include filename="$(find jackal_kinova_gazebo)/urdf/include/tim571.urdf.xacro"/>
   <xacro:include filename="$(find jackal_kinova_gazebo)/urdf/include/d435.urdf.xacro"/>
+  <xacro:include filename="$(find jackal_kinova_gazebo)/urdf/include/d435_collision.urdf.xacro"/>
   <!-- include arm urdf -->
   <xacro:include filename="$(find jackal_kinova_gazebo)/urdf/gen3_lite_gen3_lite_2f.xacro">

Commit message: Create branch

File: jackal_kinova_gazebo/urdf/gen3_lite/6dof/urdf/gen3_lite_macro.xacro (robot description, xacro)
@@ -206,5 +206,5 @@
       <limit lower="0" upper="0" effort="0" velocity="0" />
     </joint>
-  <link name="hand_camera_bracket">
+  <link name="${prefix}hand_camera_bracket">
     <visual>
       <origin xyz="-0.175 -0.01 -1.15" rpy="${PI/2} 0 ${PI/2}"/>
@@ -223,7 +223,7 @@
     </collision>
   </link>
-  <joint name="hand_camera_bracket_joint" type="fixed">
+  <joint name="${prefix}hand_camera_bracket_joint" type="fixed">
     <parent link="${prefix}end_effector_link"/>
-    <child link="hand_camera_bracket"/>
+    <child link="${prefix}hand_camera_bracket"/>
     <origin xyz="0 0 0" rpy="0 0 0"/>
   </joint>

File: jackal_kinova_gazebo/urdf/jackal_kinova.urdf.xacro (robot description, xacro)
@@ -9,4 +9,7 @@
   <xacro:include filename="$(find jackal_kinova_gazebo)/urdf/gen3_lite_gen3_lite_2f.xacro">
     <arg name="sim" value="true"/>
+  </xacro:include>
+  <!-- Bring in simulation data for Gazebo. -->
+  <xacro:include filename="$(find jackal_kinova_gazebo)/urdf/jackal.gazebo" >
   </xacro:include>
   <!-- lidar, base_camera mount -->
@@ -36,5 +39,5 @@
     <parent link="base_link"/>
     <child link="gen3_lite_base_link"/>
-    <origin xyz="0.01 0 0.214" rpy="0 0 0"/>
+    <origin xyz="0.01 0 0.25" rpy="0 0 0"/>
   </joint>
   <xacro:sensor_d435 parent="base_link" name="base_camera">

File: jackal_kinova_gazebo/urdf/jackal_with_ns.urdf.xacro (robot description, xacro)
@@ -1,4 +1,5 @@
 <?xml version="1.0"?>
 <robot name="jackal" xmlns:xacro="http://www.ros.org/wiki/xacro">
+  <xacro:arg name="ns" default="JK_01"/>
   <xacro:property name="PI" value="3.1415926535897931" />
   <xacro:property name="wheelbase" value="0.262" />
@@ -51,5 +52,5 @@
     </gazebo>
     <joint name="${prefix}_wheel" type="continuous">
-      <parent link="chassis_link"/>
+      <parent link="$(arg ns)chassis_link"/>
       <child link="${prefix}_wheel_link" />
       <xacro:insert_block name="joint_pose" />
@@ -68,23 +69,23 @@
     </transmission>
   </xacro:macro>
-  <xacro:wheel prefix="front_left">
+  <xacro:wheel prefix="$(arg ns)front_left">
     <origin xyz="${wheelbase/2} ${track/2} ${wheel_vertical_offset}" rpy="0 0 0" />
   </xacro:wheel>
-  <xacro:wheel prefix="front_right">
+  <xacro:wheel prefix="$(arg ns)front_right">
     <origin xyz="${wheelbase/2} ${-track/2} ${wheel_vertical_offset}" rpy="0 0 0" />
   </xacro:wheel>
-  <xacro:wheel prefix="rear_left">
+  <xacro:wheel prefix="$(arg ns)rear_left">
     <origin xyz="${-wheelbase/2} ${track/2} ${wheel_vertical_offset}" rpy="0 0 0" />
   </xacro:wheel>
-  <xacro:wheel prefix="rear_right">
+  <xacro:wheel prefix="$(arg ns)rear_right">
     <origin xyz="${-wheelbase/2} ${-track/2} ${wheel_vertical_offset}" rpy="0 0 0" />
   </xacro:wheel>
-  <link name="base_link"></link>
-  <joint name="base_link_joint" type="fixed">
+  <link name="$(arg ns)base_link"></link>
+  <joint name="$(arg ns)base_link_joint" type="fixed">
     <origin xyz="0 0 0" rpy="0 0 0" />
-    <parent link="base_link"/>
-    <child link="chassis_link" />
-  </joint>
-  <link name="chassis_link">
+    <parent link="$(arg ns)base_link"/>
+    <child link="$(arg ns)chassis_link" />
+  </joint>
+  <link name="$(arg ns)chassis_link">
     <visual>
       <origin xyz="0 0 ${footprint_vertical_offset}" rpy="${PI/2} 0 ${PI/2}"/>
@@ -112,5 +113,5 @@
   </link>
   <xacro:unless value="$(optenv JACKAL_FRONT_ACCESSORY_FENDER 0)">
-    <link name="front_fender_link">
+    <link name="$(arg ns)front_fender_link">
       <visual>
         <geometry>
@@ -122,5 +123,5 @@
   </xacro:unless>
   <xacro:if value="$(optenv JACKAL_FRONT_ACCESSORY_FENDER 0)">
-    <link name="front_fender_link">
+    <link name="$(arg ns)front_fender_link">
       <visual>
         <geometry>
@@ -130,18 +131,18 @@
       </visual>
     </link>
-    <link name="front_fender_accessory_link"/>
-    <joint name="front_fender_accessory_joint" type="fixed">
+    <link name="$(arg ns)front_fender_accessory_link"/>
+    <joint name="$(arg ns)front_fender_accessory_joint" type="fixed">
       <origin xyz="0.25629 0 0.07455" rpy="${PI} 0 0" />
-      <parent link="front_fender_link" />
-      <child link="front_fender_accessory_link" />
+      <parent link="$(arg ns)front_fender_link" />
+      <child link="$(arg ns)front_fender_accessory_link" />
     </joint>
   </xacro:if>
-  <joint name="front_fender_joint" type="fixed">
+  <joint name="$(arg ns)front_fender_joint" type="fixed">
     <origin xyz="0 0 0" rpy="0 0 0"/>
-    <parent link="chassis_link" />
-    <child link="front_fender_link" />
+    <parent link="$(arg ns)chassis_link" />
+    <child link="$(arg ns)front_fender_link" />
   </joint>
   <xacro:unless value="$(optenv JACKAL_REAR_ACCESSORY_FENDER 0)">
-    <link name="rear_fender_link">
+    <link name="$(arg ns)rear_fender_link">
       <visual>
         <geometry>
@@ -153,5 +154,5 @@
   </xacro:unless>
   <xacro:if value="$(optenv JACKAL_REAR_ACCESSORY_FENDER 0)">
-    <link name="rear_fender_link">
+    <link name="$(arg ns)rear_fender_link">
       <visual>
         <geometry>
@@ -161,18 +162,18 @@
       </visual>
     </link>
-    <link name="rear_fender_accessory_link"/>
-    <joint name="rear_fender_accessory_joint" type="fixed">
+    <link name="$(arg ns)rear_fender_accessory_link"/>
+    <joint name="$(arg ns)rear_fender_accessory_joint" type="fixed">
       <origin xyz="0.25629 0 0.07455" rpy="${PI} 0 0" />
-      <parent link="rear_fender_link" />
-      <child link="rear_fender_accessory_link" />
+      <parent link="$(arg ns)rear_fender_link" />
+      <child link="$(arg ns)rear_fender_accessory_link" />
     </joint>
   </xacro:if>
-  <joint name="rear_fender_joint" type="fixed">
+  <joint name="$(arg ns)rear_fender_joint" type="fixed">
     <origin xyz="0 0 0" rpy="0 0 ${PI}"/>
-    <parent link="chassis_link" />
-    <child link="rear_fender_link" />
+    <parent link="$(arg ns)chassis_link" />
+    <child link="$(arg ns)rear_fender_link" />
   </joint>
   <!-- Default Internal IMU Link -->
-  <link name="imu_link">
+  <link name="$(arg ns)imu_link">
     <inertial>
       <mass value="0.001"/>
@@ -181,10 +182,10 @@
     </inertial>
   </link>
-  <joint name="imu_joint" type="fixed">
-    <parent link="base_link" />
-    <child link="imu_link" />
+  <joint name="$(arg ns)imu_joint" type="fixed">
+    <parent link="$(arg ns)base_link" />
+    <child link="$(arg ns)imu_link" />
   </joint>
   <!-- Default NAVSAT Link -->
-  <link name="navsat_link">
+  <link name="$(arg ns)navsat_link">
     <visual>
       <geometry>
@@ -195,25 +196,25 @@
     </visual>
   </link>
-  <joint name="navsat_joint" type="fixed">
-    <parent link="base_link" />
-    <child link="navsat_link" />
+  <joint name="$(arg ns)navsat_joint" type="fixed">
+    <parent link="$(arg ns)base_link" />
+    <child link="$(arg ns)navsat_link" />
     <origin xyz="-0.180 0.126 0.1815" />
   </joint>
-  <link name="mid_mount"></link>
-  <joint name="mid_mount_joint" type="fixed">
-    <parent link="chassis_link" />
-    <child link="mid_mount" />
+  <link name="$(arg ns)mid_mount"></link>
+  <joint name="$(arg ns)mid_mount_joint" type="fixed">
+    <parent link="$(arg ns)chassis_link" />
+    <child link="$(arg ns)mid_mount" />
     <origin xyz="0 0 ${chassis_height}" />
   </joint>
-  <link name="rear_mount"></link>
-  <joint name="rear_mount_joint" type="fixed">
-    <parent link="mid_mount" />
-    <child link="rear_mount" />
+  <link name="$(arg ns)rear_mount"></link>
+  <joint name="$(arg ns)rear_mount_joint" type="fixed">
+    <parent link="$(arg ns)mid_mount" />
+    <child link="$(arg ns)rear_mount" />
     <origin xyz="${-mount_spacing} 0 0" />
   </joint>
-  <link name="front_mount"></link>
-  <joint name="front_mount_joint" type="fixed">
-    <parent link="mid_mount" />
-    <child link="front_mount" />
+  <link name="$(arg ns)front_mount"></link>
+  <joint name="$(arg ns)front_mount_joint" type="fixed">
+    <parent link="$(arg ns)mid_mount" />
+    <child link="$(arg ns)front_mount" />
     <origin xyz="${mount_spacing} 0 0" />
   </joint>
@@ -221,5 +222,5 @@
        of these into the final description is controlled by optenv variables, which
        default each one to off.-->
-  <xacro:include filename="$(find jackal_kinova_gazebo)/urdf/accessories.urdf.xacro" />
+  <!-- <xacro:include filename="$(find jackal_kinova_gazebo)/urdf/accessories.urdf.xacro" /> -->
   <!-- Optional custom includes. -->
   <xacro:include filename="$(optenv JACKAL_URDF_EXTRAS empty.urdf)" />
