Commit message: Add RL components

File: jackal_kinova_gazebo/urdf/include/m_d435.urdf.xacro (robot description, xacro)
@@ -1,46 +1,49 @@
 <?xml version="1.0"?>
 <robot xmlns:xacro="http://ros.org/wiki/xacro" name="sensor_d435">
-  <xacro:macro name="sensor_d435" params="*origin parent name:=camera use_nominal_extrinsics:=false camera">
-    <xacro:property name="M_PI" value="3.1415926535897931"/>
+  <xacro:macro name="sensor_d435"
+    params="*origin parent name:=camera use_nominal_extrinsics:=false camera">
+    <xacro:property name="M_PI" value="3.1415926535897931" />
     <!-- The following values are approximate, and the camera node
      publishing TF values with actual calibrated camera extrinsic values -->
-    <xacro:property name="d435_cam_depth_to_infra1_offset" value="0.0"/>
-    <xacro:property name="d435_cam_depth_to_infra2_offset" value="-0.050"/>
-    <xacro:property name="d435_cam_depth_to_color_offset" value="0.015"/>
+    <xacro:property name="d435_cam_depth_to_infra1_offset" value="0.0" />
+    <xacro:property name="d435_cam_depth_to_infra2_offset" value="-0.050" />
+    <xacro:property name="d435_cam_depth_to_color_offset" value="0.015" />
     <!-- The following values model the aluminum peripherial case for the
   	D435 camera, with the camera joint represented by the actual
   	peripherial camera tripod mount -->
-    <xacro:property name="d435_cam_width" value="0.090"/>
-    <xacro:property name="d435_cam_height" value="0.025"/>
-    <xacro:property name="d435_cam_depth" value="0.02505"/>
-    <xacro:property name="d435_cam_mount_from_center_offset" value="0.0149"/>
+    <xacro:property name="d435_cam_width" value="0.090" />
+    <xacro:property name="d435_cam_height" value="0.025" />
+    <xacro:property name="d435_cam_depth" value="0.02505" />
+    <xacro:property name="d435_cam_mount_from_center_offset" value="0.0149" />
     <!-- glass cover is 0.1 mm inwards from front aluminium plate -->
-    <xacro:property name="d435_glass_to_front" value="0.1e-3"/>
+    <xacro:property name="d435_glass_to_front" value="0.1e-3" />
     <!-- see datasheet Revision 007, Fig. 4-4 page 65 -->
-    <xacro:property name="d435_zero_depth_to_glass" value="4.2e-3"/>
+    <xacro:property name="d435_zero_depth_to_glass" value="4.2e-3" />
     <!-- convenience precomputation to avoid clutter-->
-    <xacro:property name="d435_mesh_x_offset" value="${d435_cam_mount_from_center_offset-d435_glass_to_front-d435_zero_depth_to_glass}"/>
+    <xacro:property name="d435_mesh_x_offset"
+      value="${d435_cam_mount_from_center_offset-d435_glass_to_front-d435_zero_depth_to_glass}" />
     <!-- The following offset is relative the the physical D435 camera peripherial
   	camera tripod mount -->
-    <xacro:property name="d435_cam_depth_px" value="${d435_cam_mount_from_center_offset}"/>
-    <xacro:property name="d435_cam_depth_py" value="0.0175"/>
-    <xacro:property name="d435_cam_depth_pz" value="${d435_cam_height/2}"/>
+    <xacro:property name="d435_cam_depth_px" value="${d435_cam_mount_from_center_offset}" />
+    <xacro:property name="d435_cam_depth_py" value="0.0175" />
+    <xacro:property name="d435_cam_depth_pz" value="${d435_cam_height/2}" />
     <!-- camera body, with origin at bottom screw mount -->
     <joint name="${name}_joint" type="fixed">
       <xacro:insert_block name="origin" />
-      <parent link="${parent}"/>
+      <parent link="${parent}" />
       <child link="${name}_bottom_screw_frame" />
     </joint>
-    <link name="${name}_bottom_screw_frame"/>
+    <link name="${name}_bottom_screw_frame" />
     <joint name="${name}_link_joint" type="fixed">
-      <origin xyz="${d435_mesh_x_offset} ${d435_cam_depth_py} ${d435_cam_depth_pz}" rpy="0 0 0"/>
-      <parent link="${name}_bottom_screw_frame"/>
+      <origin xyz="${d435_mesh_x_offset} ${d435_cam_depth_py} ${d435_cam_depth_pz}" rpy="0 0 0" />
+      <parent link="${name}_bottom_screw_frame" />
       <child link="${name}_link" />
     </joint>
     <link name="${name}_link">
       <visual>
-        <origin xyz="${d435_zero_depth_to_glass + d435_glass_to_front} ${-d435_cam_depth_py} 0" rpy="${M_PI/2} 0 ${M_PI/2}"/>
+        <origin xyz="${d435_zero_depth_to_glass + d435_glass_to_front} ${-d435_cam_depth_py} 0"
+          rpy="${M_PI/2} 0 ${M_PI/2}" />
         <geometry>
-          <mesh filename="package://jackal_kinova_gazebo/meshes/include/d435.dae"/>
+          <mesh filename="package://jackal_kinova_gazebo/meshes/include/d435.dae" />
         </geometry>
       </visual>
@@ -50,14 +53,21 @@
         <inertia ixx="0.003881243" ixy="0.0" ixz="0.0" iyy="0.000498940" iyz="0.0" izz="0.003879257" />
       </inertial>
+      <collision>
+        <origin xyz="0 ${-d435_cam_depth_py} 0" rpy="0 0 0" />
+        <geometry>
+          <box size="${d435_cam_depth} ${d435_cam_width} ${d435_cam_height}" />
+        </geometry>
+      </collision>
     </link>
-    <!-- Use the nominal extrinsics between camera frames if the calibrated extrinsics aren't being published. e.g. running the device in simulation  -->
+    <!-- Use the nominal extrinsics between camera frames if the calibrated extrinsics aren't being
+    published. e.g. running the device in simulation  -->
     <xacro:if value="${use_nominal_extrinsics}">
       <!-- camera depth joints and links -->
       <joint name="${name}_depth_joint" type="fixed">
-        <origin xyz="0 0 0" rpy="0 0 0"/>
-        <parent link="${name}_link"/>
+        <origin xyz="0 0 0" rpy="0 0 0" />
+        <parent link="${name}_link" />
         <child link="${name}_depth_frame" />
       </joint>
-      <link name="${name}_depth_frame"/>
+      <link name="${name}_depth_frame" />
       <joint name="${name}_depth_optical_joint" type="fixed">
         <origin xyz="0 0 0" rpy="${-M_PI/2} 0 ${-M_PI/2}" />
@@ -65,5 +75,5 @@
         <child link="${name}_depth_optical_frame" />
       </joint>
-      <link name="${name}_depth_optical_frame"/>
+      <link name="${name}_depth_optical_frame" />
       <!-- camera left IR joints and links -->
       <joint name="${name}_infra1_joint" type="fixed">
@@ -72,5 +82,5 @@
         <child link="${name}_infra1_frame" />
       </joint>
-      <link name="${name}_infra1_frame"/>
+      <link name="${name}_infra1_frame" />
       <joint name="${name}_infra1_optical_joint" type="fixed">
         <origin xyz="0 0 0" rpy="${-M_PI/2} 0 ${-M_PI/2}" />
@@ -78,5 +88,5 @@
         <child link="${name}_infra1_optical_frame" />
       </joint>
-      <link name="${name}_infra1_optical_frame"/>
+      <link name="${name}_infra1_optical_frame" />
       <!-- camera right IR joints and links -->
       <joint name="${name}_infra2_joint" type="fixed">
@@ -85,5 +95,5 @@
         <child link="${name}_infra2_frame" />
       </joint>
-      <link name="${name}_infra2_frame"/>
+      <link name="${name}_infra2_frame" />
       <joint name="${name}_infra2_optical_joint" type="fixed">
         <origin xyz="0 0 0" rpy="${-M_PI/2} 0 ${-M_PI/2}" />
@@ -91,5 +101,5 @@
         <child link="${name}_infra2_optical_frame" />
       </joint>
-      <link name="${name}_infra2_optical_frame"/>
+      <link name="${name}_infra2_optical_frame" />
       <!-- camera color joints and links -->
       <joint name="${name}_color_joint" type="fixed">
@@ -98,5 +108,5 @@
         <child link="${name}_color_frame" />
       </joint>
-      <link name="${name}_color_frame"/>
+      <link name="${name}_color_frame" />
       <joint name="${name}_color_optical_joint" type="fixed">
         <origin xyz="0 0 0" rpy="${-M_PI/2} 0 ${-M_PI/2}" />
@@ -104,13 +114,13 @@
         <child link="${name}_color_optical_frame" />
       </joint>
-      <link name="${name}_color_optical_frame"/>
+      <link name="${name}_color_optical_frame" />
     </xacro:if>
     <!-- camera depth joints and links -->
     <joint name="${name}_depth_joint" type="fixed">
-      <origin xyz="0 0 0" rpy="0 0 0"/>
-      <parent link="${name}_link"/>
+      <origin xyz="0 0 0" rpy="0 0 0" />
+      <parent link="${name}_link" />
       <child link="${name}_depth_frame" />
     </joint>
-    <link name="${name}_depth_frame"/>
+    <link name="${name}_depth_frame" />
     <joint name="${name}_depth_optical_joint" type="fixed">
       <origin xyz="0 0 0" rpy="${-M_PI/2} 0 ${-M_PI/2}" />
@@ -118,5 +128,5 @@
       <child link="${name}_depth_optical_frame" />
     </joint>
-    <link name="${name}_depth_optical_frame"/>
+    <link name="${name}_depth_optical_frame" />
     <!-- camera left IR joints and links -->
     <joint name="${name}_infra1_joint" type="fixed">
@@ -125,5 +135,5 @@
       <child link="${name}_infra1_frame" />
     </joint>
-    <link name="${name}_infra1_frame"/>
+    <link name="${name}_infra1_frame" />
     <joint name="${name}_infra1_optical_joint" type="fixed">
       <origin xyz="0 0 0" rpy="${-M_PI/2} 0 ${-M_PI/2}" />
@@ -131,5 +141,5 @@
       <child link="${name}_infra1_optical_frame" />
     </joint>
-    <link name="${name}_infra1_optical_frame"/>
+    <link name="${name}_infra1_optical_frame" />
     <!-- camera right IR joints and links -->
     <joint name="${name}_infra2_joint" type="fixed">
@@ -138,5 +148,5 @@
       <child link="${name}_infra2_frame" />
     </joint>
-    <link name="${name}_infra2_frame"/>
+    <link name="${name}_infra2_frame" />
     <joint name="${name}_infra2_optical_joint" type="fixed">
       <origin xyz="0 0 0" rpy="${-M_PI/2} 0 ${-M_PI/2}" />
@@ -144,5 +154,5 @@
       <child link="${name}_infra2_optical_frame" />
     </joint>
-    <link name="${name}_infra2_optical_frame"/>
+    <link name="${name}_infra2_optical_frame" />
     <!-- camera color joints and links -->
     <joint name="${name}_color_joint" type="fixed">
@@ -151,5 +161,5 @@
       <child link="${name}_color_frame" />
     </joint>
-    <link name="${name}_color_frame"/>
+    <link name="${name}_color_frame" />
     <joint name="${name}_color_optical_joint" type="fixed">
       <origin xyz="0 0 0" rpy="${-M_PI/2} 0 ${-M_PI/2}" />
@@ -157,80 +167,80 @@
       <child link="${name}_color_optical_frame" />
     </joint>
-    <link name="${name}_color_optical_frame"/>
-  <link name="${name}_gazebo" />
-  <joint name="${name}_gazebo_joint" type="fixed">
-    <parent link="${name}_link"/>
-    <child link="${name}_gazebo"/>
-    <origin xyz="0.0 0 0" rpy="0 0 0"/>
-  </joint>
-  <gazebo reference="${name}_link">
-    <sensor name="${name}color" type="camera">
-      <camera name="${camera}">
-        <horizontal_fov>${1.211259}</horizontal_fov>
-        <image>
-          <width>640</width>
-          <height>480</height>
-          <format>RGB_INT8</format>
-        </image>
-        <clip>
-          <near>0.1</near>
-          <far>100</far>
-        </clip>
-        <noise>
-          <type>gaussian</type>
-          <mean>0.0</mean>
-          <stddev>0.007</stddev>
-        </noise>
-      </camera>
-      <always_on>0</always_on>
-      <update_rate>30</update_rate>
-      <visualize>0</visualize>
-    </sensor>
-    <turnGravityOff>true</turnGravityOff>
-    <always_on>false</always_on>
-    <visualize>false</visualize>
-    <sensor type="depth" name="${name}_gazebo_depth">
-      <update_rate>30</update_rate>
-      <camera>
-        <!-- 75x65 degree FOV for the depth sensor -->
-        <horizontal_fov>1.5184351666666667</horizontal_fov>
-        <vertical_fov>1.0122901111111111</vertical_fov>
-        <image>
-          <width>640</width>
-          <height>480</height>
-          <format>RGB_INT8</format>
-        </image>
-        <clip>
-          <!-- give the color sensor a maximum range of 50m so that the simulation renders nicely -->
-          <near>0.01</near>
-          <far>50.0</far>
-        </clip>
-      </camera>
-      <plugin name="kinect_controller" filename="libgazebo_ros_openni_kinect.so">
-        <baseline>0.2</baseline>
-        <alwaysOn>false</alwaysOn>
-        <updateRate>30</updateRate>
-        <cameraName>${camera}</cameraName>
-        <imageTopicName>color/image_raw</imageTopicName>
-        <cameraInfoTopicName>color/camera_info</cameraInfoTopicName>
-        <depthImageTopicName>depth/image_raw</depthImageTopicName>
-        <depthImageInfoTopicName>depth/camera_info</depthImageInfoTopicName>
-        <pointCloudTopicName>depth/color/points</pointCloudTopicName>
-        <frameName>${name}_depth_optical_frame</frameName>
-        <pointCloudCutoff>0.105</pointCloudCutoff>
-        <pointCloudCutoffMax>8.0</pointCloudCutoffMax>
-        <distortionK1>0.00000001</distortionK1>
-        <distortionK2>0.00000001</distortionK2>
-        <distortionK3>0.00000001</distortionK3>
-        <distortionT1>0.00000001</distortionT1>
-        <distortionT2>0.00000001</distortionT2>
-        <CxPrime>0</CxPrime>
-        <Cx>0</Cx>
-        <Cy>0</Cy>
-        <focalLength>0</focalLength>
-        <hackBaseline>0</hackBaseline>
-      </plugin>
-    </sensor>
-  </gazebo>
+    <link name="${name}_color_optical_frame" />
+    <link name="${name}_gazebo" />
+    <joint name="${name}_gazebo_joint" type="fixed">
+      <parent link="${name}_link" />
+      <child link="${name}_gazebo" />
+      <origin xyz="0.0 0 0" rpy="0 0 0" />
+    </joint>
+    <gazebo reference="${name}_link">
+      <sensor name="${name}color" type="camera">
+        <camera name="${camera}">
+          <horizontal_fov>${1.211259}</horizontal_fov>
+          <image>
+            <width>640</width>
+            <height>480</height>
+            <format>RGB_INT8</format>
+          </image>
+          <clip>
+            <near>0.1</near>
+            <far>100</far>
+          </clip>
+          <noise>
+            <type>gaussian</type>
+            <mean>0.0</mean>
+            <stddev>0.007</stddev>
+          </noise>
+        </camera>
+        <always_on>0</always_on>
+        <update_rate>30</update_rate>
+        <visualize>0</visualize>
+      </sensor>
+      <turnGravityOff>true</turnGravityOff>
+      <always_on>false</always_on>
+      <visualize>false</visualize>
+      <sensor type="depth" name="${name}_gazebo_depth">
+        <update_rate>30</update_rate>
+        <camera>
+          <!-- 75x65 degree FOV for the depth sensor -->
+          <horizontal_fov>1.5184351666666667</horizontal_fov>
+          <vertical_fov>1.0122901111111111</vertical_fov>
+          <image>
+            <width>640</width>
+            <height>480</height>
+            <format>RGB_INT8</format>
+          </image>
+          <clip>
+            <!-- give the color sensor a maximum range of 50m so that the simulation renders nicely -->
+            <near>0.01</near>
+            <far>50.0</far>
+          </clip>
+        </camera>
+        <plugin name="kinect_controller" filename="libgazebo_ros_openni_kinect.so">
+          <baseline>0.2</baseline>
+          <alwaysOn>false</alwaysOn>
+          <updateRate>30</updateRate>
+          <cameraName>${camera}</cameraName>
+          <imageTopicName>color/image_raw</imageTopicName>
+          <cameraInfoTopicName>color/camera_info</cameraInfoTopicName>
+          <depthImageTopicName>depth/image_raw</depthImageTopicName>
+          <depthImageInfoTopicName>depth/camera_info</depthImageInfoTopicName>
+          <pointCloudTopicName>depth/color/points</pointCloudTopicName>
+          <frameName>${name}_depth_optical_frame</frameName>
+          <pointCloudCutoff>0.105</pointCloudCutoff>
+          <pointCloudCutoffMax>8.0</pointCloudCutoffMax>
+          <distortionK1>0.00000001</distortionK1>
+          <distortionK2>0.00000001</distortionK2>
+          <distortionK3>0.00000001</distortionK3>
+          <distortionT1>0.00000001</distortionT1>
+          <distortionT2>0.00000001</distortionT2>
+          <CxPrime>0</CxPrime>
+          <Cx>0</Cx>
+          <Cy>0</Cy>
+          <focalLength>0</focalLength>
+          <hackBaseline>0</hackBaseline>
+        </plugin>
+      </sensor>
+    </gazebo>
   </xacro:macro>
 </robot>

File: jackal_kinova_gazebo/urdf/include/m_tim571.urdf.xacro (robot description, xacro)
@@ -1,29 +1,32 @@
 <?xml version="1.0"?>
 <robot xmlns:xacro="http://www.ros.org/wiki/xacro" name="sensor_tim571">
-  <xacro:macro name="sensor_tim571" params="*origin parent name:=laser topic:=/scan length:=0.06 width:=0.06 height:=0.079 mass:=0.15 min_angle:=-2.35619449019 max_angle:=2.35619449019 min_range:=0.05 max_range:=25.0 samples:=811 ns">
+  <xacro:macro name="sensor_tim571"
+    params="*origin parent name:=laser topic:=/scan length:=0.06 width:=0.06 height:=0.079 mass:=0.15 min_angle:=-2.35619449019 max_angle:=2.35619449019 min_range:=0.05 max_range:=25.0 samples:=811 ns">
     <joint name="${name}_base_joint" type="fixed">
-      <xacro:insert_block name="origin"/>
-      <parent link="${parent}"/>
-      <child link="${name}_base_link"/>
+      <xacro:insert_block name="origin" />
+      <parent link="${parent}" />
+      <child link="${name}_base_link" />
     </joint>
     <link name="${name}_base_link">
       <inertial>
-        <mass value="${mass}"/>
-        <origin xyz="0 0 -0.026" rpy="3.1415926 0 0"/>
-        <inertia ixx="${0.0833333 * mass * (width * width + height * height)}" ixy="0.0" ixz="0.0" iyy="${0.0833333 * mass * (length * length + height * height)}" iyz="0.0" izz="${0.0833333 * mass * (length * length + width * width)}" />
+        <mass value="${mass}" />
+        <origin xyz="0 0 -0.026" rpy="3.1415926 0 0" />
+        <inertia ixx="${0.0833333 * mass * (width * width + height * height)}" ixy="0.0" ixz="0.0"
+          iyy="${0.0833333 * mass * (length * length + height * height)}" iyz="0.0"
+          izz="${0.0833333 * mass * (length * length + width * width)}" />
       </inertial>
     </link>
     <joint name="${name}_joint" type="fixed">
-      <origin xyz="0 0 -0.06246" rpy="0 0 0"/>
-      <parent link="${name}_base_link"/>
-      <child link="${name}_link"/>
+      <origin xyz="0 0 -0.06246" rpy="0 0 0" />
+      <parent link="${name}_base_link" />
+      <child link="${name}_link" />
     </joint>
     <link name="${name}_link">
     </link>
-    <xacro:tim571_gazebo/>
+    <xacro:tim571_gazebo />
   </xacro:macro>
   <xacro:macro name="tim571_gazebo">
     <gazebo reference="${name}_link">
-      <material value="Gazebo/Blue"/>
+      <material value="Gazebo/Blue" />
       <sensor type="ray" name="${name}">
         <always_on>true</always_on>
@@ -45,9 +48,9 @@
             <resolution>0.01</resolution>
           </range>
-					<noise>
-						<type>gaussian</type>
-						<mean>0.0</mean>
-						<stddev>0.01</stddev>
-					</noise>
+          <noise>
+            <type>gaussian</type>
+            <mean>0.0</mean>
+            <stddev>0.01</stddev>
+          </noise>
         </ray>
         <plugin name="gazebo_ros_laser_controller" filename="libgazebo_ros_laser.so">
