Commit message: Add RL components

File: jackal_kinova_gazebo/urdf/jackal_with_ns.urdf.xacro (robot description, xacro)
@@ -1,5 +1,5 @@
 <?xml version="1.0"?>
 <robot name="jackal" xmlns:xacro="http://www.ros.org/wiki/xacro">
-  <xacro:arg name="ns" default="JK_01"/>
+  <xacro:arg name="ns" default="JK_01" />
   <xacro:property name="PI" value="3.1415926535897931" />
   <xacro:property name="wheelbase" value="0.262" />
@@ -12,32 +12,40 @@
   <xacro:property name="chassis_width" value="0.310" />
   <xacro:property name="chassis_height" value="0.184" />
-  <xacro:property name="dummy_inertia" value="1e-09"/>
+  <xacro:property name="dummy_inertia" value="1e-09" />
   <xacro:property name="mount_spacing" value="0.120" />
-  <material name="dark_grey"><color rgba="0.2 0.2 0.2 1.0" /></material>
-  <material name="light_grey"><color rgba="0.4 0.4 0.4 1.0" /></material>
-  <material name="yellow"><color rgba="0.8 0.8 0.0 1.0" /></material>
-  <material name="black"><color rgba="0.15 0.15 0.15 1.0" /></material>
+  <material name="dark_grey">
+    <color rgba="0.2 0.2 0.2 1.0" />
+  </material>
+  <material name="light_grey">
+    <color rgba="0.4 0.4 0.4 1.0" />
+  </material>
+  <material name="yellow">
+    <color rgba="0.8 0.8 0.0 1.0" />
+  </material>
+  <material name="black">
+    <color rgba="0.15 0.15 0.15 1.0" />
+  </material>
   <xacro:macro name="wheel" params="prefix *joint_pose">
     <link name="${prefix}_wheel_link">
       <visual>
-        <origin xyz="0 0 0" rpy="${PI/2} 0 0"/>
-        <geometry>
-          <mesh filename="package://jackal_kinova_gazebo/meshes/jackal-wheel.stl"/>
+        <origin xyz="0 0 0" rpy="${PI/2} 0 0" />
+        <geometry>
+          <mesh filename="package://jackal_kinova_gazebo/meshes/jackal-wheel.stl" />
         </geometry>
         <material name="black" />
       </visual>
       <collision>
-        <origin xyz="0 0 0" rpy="${PI/2} 0 0"/>
-        <geometry>
-          <cylinder radius="${wheel_radius}" length="${wheel_width}"/>
+        <origin xyz="0 0 0" rpy="${PI/2} 0 0" />
+        <geometry>
+          <cylinder radius="${wheel_radius}" length="${wheel_width}" />
         </geometry>
       </collision>
       <inertial>
-        <origin xyz="0 0 0" rpy="0 0 0"/>
-        <mass value="0.477"/>
+        <origin xyz="0 0 0" rpy="0 0 0" />
+        <mass value="0.477" />
         <inertia
           ixx="0.0013" ixy="0" ixz="0"
           iyy="0.0024" iyz="0"
-          izz="0.0013"/>
+          izz="0.0013" />
       </inertial>
     </link>
@@ -45,12 +53,12 @@
       <material>Gazebo/DarkGrey</material>
       <selfCollide>false</selfCollide>
-      <mu1 value="0.75"/>
-      <mu2 value="0.75"/>
+      <mu1 value="0.75" />
+      <mu2 value="0.75" />
       <kp value="10000000.0" />
       <kd value="1" />
-      <fdir1 value="1 0 0"/>
+      <fdir1 value="1 0 0" />
     </gazebo>
     <joint name="${prefix}_wheel" type="continuous">
-      <parent link="$(arg ns)chassis_link"/>
+      <parent link="$(arg ns)chassis_link" />
       <child link="${prefix}_wheel_link" />
       <xacro:insert_block name="joint_pose" />
@@ -84,31 +92,25 @@
   <joint name="$(arg ns)base_link_joint" type="fixed">
     <origin xyz="0 0 0" rpy="0 0 0" />
-    <parent link="$(arg ns)base_link"/>
+    <parent link="$(arg ns)base_link" />
     <child link="$(arg ns)chassis_link" />
   </joint>
   <link name="$(arg ns)chassis_link">
     <visual>
-      <origin xyz="0 0 ${footprint_vertical_offset}" rpy="${PI/2} 0 ${PI/2}"/>
+      <origin xyz="0 0 ${footprint_vertical_offset}" rpy="${PI/2} 0 ${PI/2}" />
       <geometry>
-        <mesh filename="package://jackal_kinova_gazebo/meshes/jackal-base.stl"/>
+        <mesh filename="package://jackal_kinova_gazebo/meshes/jackal-base.stl" />
       </geometry>
       <material name="dark_grey" />
     </visual>
-    <collision>
-      <origin xyz="0 0 ${chassis_height/2}"/>
-      <geometry>
-        <box size="${chassis_length} ${chassis_width} ${chassis_height}"/>
-      </geometry>
-    </collision>
     <inertial>
       <!-- Center of mass -->
-      <origin xyz="0.012  0.002 0.067" rpy="0 0 0"/>
-      <mass value="16.523"/>
+      <origin xyz="0.012  0.002 0.067" rpy="0 0 0" />
+      <mass value="16.523" />
       <!-- Moments of inertia: ( chassis without wheels ) -->
       <inertia
         ixx="0.3136" ixy="-0.0008" ixz="0.0164"
         iyy="0.3922" iyz="-0.0009"
-        izz="0.4485"/>
-      </inertial>
+        izz="0.4485" />
+    </inertial>
   </link>
   <xacro:unless value="$(optenv JACKAL_FRONT_ACCESSORY_FENDER 0)">
@@ -116,8 +118,14 @@
       <visual>
         <geometry>
-          <mesh filename="package://jackal_kinova_gazebo/meshes/jackal-fender.stl"/>
-        </geometry>
-        <material name="yellow" />
-      </visual>
+          <mesh filename="package://jackal_kinova_gazebo/meshes/jackal-fender.stl" />
+        </geometry>
+        <material name="yellow" />
+      </visual>
+      <collision name="$(arg ns)front_fender_collision">
+        <geometry>
+          <mesh filename="package://jackal_kinova_gazebo/meshes/jackal-fender.stl"
+            scale="1.2 1.2 1.0" />
+        </geometry>
+      </collision>
     </link>
   </xacro:unless>
@@ -126,10 +134,16 @@
       <visual>
         <geometry>
-          <mesh filename="package://jackal_kinova_gazebo/meshes/accessory_fender.stl"/>
-        </geometry>
-        <material name="yellow" />
-      </visual>
-    </link>
-    <link name="$(arg ns)front_fender_accessory_link"/>
+          <mesh filename="package://jackal_kinova_gazebo/meshes/accessory_fender.stl" />
+        </geometry>
+        <material name="yellow" />
+      </visual>
+      <collision name="$(arg ns)front_fender_collision">
+        <geometry>
+          <mesh filename="package://jackal_kinova_gazebo/meshes/accessory_fender.stl"
+            scale="1.2 1.2 1.0" />
+        </geometry>
+      </collision>
+    </link>
+    <link name="$(arg ns)front_fender_accessory_link" />
     <joint name="$(arg ns)front_fender_accessory_joint" type="fixed">
       <origin xyz="0.25629 0 0.07455" rpy="${PI} 0 0" />
@@ -139,5 +153,5 @@
   </xacro:if>
   <joint name="$(arg ns)front_fender_joint" type="fixed">
-    <origin xyz="0 0 0" rpy="0 0 0"/>
+    <origin xyz="0 0 0" rpy="0 0 0" />
     <parent link="$(arg ns)chassis_link" />
     <child link="$(arg ns)front_fender_link" />
@@ -147,8 +161,14 @@
       <visual>
         <geometry>
-          <mesh filename="package://jackal_kinova_gazebo/meshes/jackal-fender.stl"/>
-        </geometry>
-        <material name="yellow" />
-      </visual>
+          <mesh filename="package://jackal_kinova_gazebo/meshes/jackal-fender.stl" />
+        </geometry>
+        <material name="yellow" />
+      </visual>
+      <collision name="$(arg ns)rear_fender_collision">
+        <geometry>
+          <mesh filename="package://jackal_kinova_gazebo/meshes/jackal-fender.stl"
+            scale="1.2 1.2 1.0" />
+        </geometry>
+      </collision>
     </link>
   </xacro:unless>
@@ -157,10 +177,16 @@
       <visual>
         <geometry>
-          <mesh filename="package://jackal_kinova_gazebo/meshes/accessory_fender.stl"/>
-        </geometry>
-        <material name="yellow" />
-      </visual>
-    </link>
-    <link name="$(arg ns)rear_fender_accessory_link"/>
+          <mesh filename="package://jackal_kinova_gazebo/meshes/accessory_fender.stl" />
+        </geometry>
+        <material name="yellow" />
+      </visual>
+      <collision name="$(arg ns)rear_fender_collision">
+        <geometry>
+          <mesh filename="package://jackal_kinova_gazebo/meshes/jackal-fender.stl"
+            scale="1.2 1.2 1.0" />
+        </geometry>
+      </collision>
+    </link>
+    <link name="$(arg ns)rear_fender_accessory_link" />
     <joint name="$(arg ns)rear_fender_accessory_joint" type="fixed">
       <origin xyz="0.25629 0 0.07455" rpy="${PI} 0 0" />
@@ -170,5 +196,5 @@
   </xacro:if>
   <joint name="$(arg ns)rear_fender_joint" type="fixed">
-    <origin xyz="0 0 0" rpy="0 0 ${PI}"/>
+    <origin xyz="0 0 0" rpy="0 0 ${PI}" />
     <parent link="$(arg ns)chassis_link" />
     <child link="$(arg ns)rear_fender_link" />
@@ -177,7 +203,8 @@
   <link name="$(arg ns)imu_link">
     <inertial>
-      <mass value="0.001"/>
-      <origin xyz="0 0 0" rpy="0 0 0"/>
-      <inertia ixx="${dummy_inertia}" ixy="0.0" ixz="0.0" iyy="${dummy_inertia}" iyz="0.0" izz="${dummy_inertia}"/>
+      <mass value="0.001" />
+      <origin xyz="0 0 0" rpy="0 0 0" />
+      <inertia ixx="${dummy_inertia}" ixy="0.0" ixz="0.0" iyy="${dummy_inertia}" iyz="0.0"
+        izz="${dummy_inertia}" />
     </inertial>
   </link>
