Commit message: Add non-ns env

File: jackal_kinova_gazebo/urdf/include/tim571.urdf.xacro (robot description, xacro)
@@ -1,30 +1,33 @@
 <?xml version="1.0"?>
 <robot xmlns:xacro="http://www.ros.org/wiki/xacro" name="sensor_tim571">
-  <xacro:macro name="sensor_tim571" params="*origin parent name:=laser topic:=/scan length:=0.06 width:=0.06 height:=0.079 mass:=0.15 min_angle:=-2.35619449019 max_angle:=2.35619449019 min_range:=0.05 max_range:=25.0 samples:=811 ">
+  <xacro:macro name="sensor_tim571"
+    params="*origin parent name:=laser topic:=/scan length:=0.06 width:=0.06 height:=0.079 mass:=0.15 min_angle:=-2.35619449019 max_angle:=2.35619449019 min_range:=0.05 max_range:=25.0 samples:=811 ">
     <joint name="${name}_base_joint" type="fixed">
-      <xacro:insert_block name="origin"/>
-      <parent link="${parent}"/>
-      <child link="${name}_base_link"/>
+      <xacro:insert_block name="origin" />
+      <parent link="${parent}" />
+      <child link="${name}_base_link" />
     </joint>
     <link name="${name}_base_link">
       <inertial>
-        <mass value="${mass}"/>
-        <origin xyz="0 0 -0.026" rpy="3.1415926 0 0"/>
-        <inertia ixx="${0.0833333 * mass * (width * width + height * height)}" ixy="0.0" ixz="0.0" iyy="${0.0833333 * mass * (length * length + height * height)}" iyz="0.0" izz="${0.0833333 * mass * (length * length + width * width)}" />
+        <mass value="${mass}" />
+        <origin xyz="0 0 -0.026" rpy="3.1415926 0 0" />
+        <inertia ixx="${0.0833333 * mass * (width * width + height * height)}" ixy="0.0" ixz="0.0"
+          iyy="${0.0833333 * mass * (length * length + height * height)}" iyz="0.0"
+          izz="${0.0833333 * mass * (length * length + width * width)}" />
       </inertial>
     </link>
     <joint name="${name}_joint" type="fixed">
-      <origin xyz="0 0 -0.06246" rpy="0 0 0"/>
-      <parent link="${name}_base_link"/>
-      <child link="${name}_link"/>
+      <origin xyz="0 0 -0.06246" rpy="0 0 0" />
+      <parent link="${name}_base_link" />
+      <child link="${name}_link" />
     </joint>
     <link name="${name}_link">
     </link>
-    <xacro:tim571_gazebo/>
+    <xacro:tim571_gazebo />
   </xacro:macro>
   <xacro:macro name="tim571_gazebo">
     <gazebo reference="${name}_link">
-      <material value="Gazebo/Blue"/>
-      <sensor type="ray" name="${name}">
+      <material value="Gazebo/Blue" />
+      <sensor type="gpu_ray" name="${name}">
         <always_on>true</always_on>
         <update_rate>15.0</update_rate>
@@ -45,9 +48,9 @@
             <resolution>0.01</resolution>
           </range>
-					<noise>
-						<type>gaussian</type>
-						<mean>0.0</mean>
-						<stddev>0.01</stddev>
-					</noise>
+          <noise>
+            <type>gaussian</type>
+            <mean>0.0</mean>
+            <stddev>0.01</stddev>
+          </noise>
         </ray>
         <plugin name="gazebo_ros_laser_controller" filename="libgazebo_ros_laser.so">

File: jackal_kinova_gazebo/urdf/jackal.urdf.xacro (robot description, xacro)
@@ -11,32 +11,40 @@
   <xacro:property name="chassis_width" value="0.310" />
   <xacro:property name="chassis_height" value="0.184" />
-  <xacro:property name="dummy_inertia" value="1e-09"/>
+  <xacro:property name="dummy_inertia" value="1e-09" />
   <xacro:property name="mount_spacing" value="0.120" />
-  <material name="dark_grey"><color rgba="0.2 0.2 0.2 1.0" /></material>
-  <material name="light_grey"><color rgba="0.4 0.4 0.4 1.0" /></material>
-  <material name="yellow"><color rgba="0.8 0.8 0.0 1.0" /></material>
-  <material name="black"><color rgba="0.15 0.15 0.15 1.0" /></material>
+  <material name="dark_grey">
+    <color rgba="0.2 0.2 0.2 1.0" />
+  </material>
+  <material name="light_grey">
+    <color rgba="0.4 0.4 0.4 1.0" />
+  </material>
+  <material name="yellow">
+    <color rgba="0.8 0.8 0.0 1.0" />
+  </material>
+  <material name="black">
+    <color rgba="0.15 0.15 0.15 1.0" />
+  </material>
   <xacro:macro name="wheel" params="prefix *joint_pose">
     <link name="${prefix}_wheel_link">
       <visual>
-        <origin xyz="0 0 0" rpy="${PI/2} 0 0"/>
-        <geometry>
-          <mesh filename="package://jackal_kinova_gazebo/meshes/jackal-wheel.stl"/>
+        <origin xyz="0 0 0" rpy="${PI/2} 0 0" />
+        <geometry>
+          <mesh filename="package://jackal_kinova_gazebo/meshes/jackal-wheel.stl" />
         </geometry>
         <material name="black" />
       </visual>
       <collision>
-        <origin xyz="0 0 0" rpy="${PI/2} 0 0"/>
-        <geometry>
-          <cylinder radius="${wheel_radius}" length="${wheel_width}"/>
+        <origin xyz="0 0 0" rpy="${PI/2} 0 0" />
+        <geometry>
+          <cylinder radius="${wheel_radius}" length="${wheel_width}" />
         </geometry>
       </collision>
       <inertial>
-        <origin xyz="0 0 0" rpy="0 0 0"/>
-        <mass value="0.477"/>
+        <origin xyz="0 0 0" rpy="0 0 0" />
+        <mass value="0.477" />
         <inertia
           ixx="0.0013" ixy="0" ixz="0"
           iyy="0.0024" iyz="0"
-          izz="0.0013"/>
+          izz="0.0013" />
       </inertial>
     </link>
@@ -44,12 +52,12 @@
       <material>Gazebo/DarkGrey</material>
       <selfCollide>false</selfCollide>
-      <mu1 value="0.75"/>
-      <mu2 value="0.75"/>
+      <mu1 value="0.75" />
+      <mu2 value="0.75" />
       <kp value="10000000.0" />
       <kd value="1" />
-      <fdir1 value="1 0 0"/>
+      <fdir1 value="1 0 0" />
     </gazebo>
     <joint name="${prefix}_wheel" type="continuous">
-      <parent link="chassis_link"/>
+      <parent link="chassis_link" />
       <child link="${prefix}_wheel_link" />
       <xacro:insert_block name="joint_pose" />
@@ -83,31 +91,31 @@
   <joint name="base_link_joint" type="fixed">
     <origin xyz="0 0 0" rpy="0 0 0" />
-    <parent link="base_link"/>
+    <parent link="base_link" />
     <child link="chassis_link" />
   </joint>
   <link name="chassis_link">
     <visual>
-      <origin xyz="0 0 ${footprint_vertical_offset}" rpy="${PI/2} 0 ${PI/2}"/>
+      <origin xyz="0 0 ${footprint_vertical_offset}" rpy="${PI/2} 0 ${PI/2}" />
       <geometry>
-        <mesh filename="package://jackal_kinova_gazebo/meshes/jackal-base.stl"/>
+        <mesh filename="package://jackal_kinova_gazebo/meshes/jackal-base.stl" />
       </geometry>
       <material name="dark_grey" />
     </visual>
     <collision>
-      <origin xyz="0 0 ${chassis_height/2}"/>
+      <origin xyz="0 0 ${chassis_height/2}" />
       <geometry>
-        <box size="${chassis_length} ${chassis_width} ${chassis_height}"/>
+        <box size="${chassis_length} ${chassis_width} ${chassis_height}" />
       </geometry>
     </collision>
     <inertial>
       <!-- Center of mass -->
-      <origin xyz="0.012  0.002 0.067" rpy="0 0 0"/>
-      <mass value="16.523"/>
+      <origin xyz="0.012  0.002 0.067" rpy="0 0 0" />
+      <mass value="16.523" />
       <!-- Moments of inertia: ( chassis without wheels ) -->
       <inertia
         ixx="0.3136" ixy="-0.0008" ixz="0.0164"
         iyy="0.3922" iyz="-0.0009"
-        izz="0.4485"/>
-      </inertial>
+        izz="0.4485" />
+    </inertial>
   </link>
   <xacro:unless value="$(optenv JACKAL_FRONT_ACCESSORY_FENDER 0)">
@@ -115,5 +123,5 @@
       <visual>
         <geometry>
-          <mesh filename="package://jackal_kinova_gazebo/meshes/jackal-fender.stl"/>
+          <mesh filename="package://jackal_kinova_gazebo/meshes/jackal-fender.stl" />
         </geometry>
         <material name="yellow" />
@@ -125,10 +133,16 @@
       <visual>
         <geometry>
-          <mesh filename="package://jackal_kinova_gazebo/meshes/accessory_fender.stl"/>
-        </geometry>
-        <material name="yellow" />
-      </visual>
-    </link>
-    <link name="front_fender_accessory_link"/>
+          <mesh filename="package://jackal_kinova_gazebo/meshes/accessory_fender.stl" />
+        </geometry>
+        <material name="yellow" />
+      </visual>
+      <collision name="front_fender_collision">
+        <geometry>
+          <mesh filename="package://jackal_kinova_gazebo/meshes/jackal-fender.stl"
+            scale="1.2 1.2 1.0" />
+        </geometry>
+      </collision>
+    </link>
+    <link name="front_fender_accessory_link" />
     <joint name="front_fender_accessory_joint" type="fixed">
       <origin xyz="0.25629 0 0.07455" rpy="${PI} 0 0" />
@@ -138,5 +152,5 @@
   </xacro:if>
   <joint name="front_fender_joint" type="fixed">
-    <origin xyz="0 0 0" rpy="0 0 0"/>
+    <origin xyz="0 0 0" rpy="0 0 0" />
     <parent link="chassis_link" />
     <child link="front_fender_link" />
@@ -146,8 +160,14 @@
       <visual>
         <geometry>
-          <mesh filename="package://jackal_kinova_gazebo/meshes/jackal-fender.stl"/>
-        </geometry>
-        <material name="yellow" />
-      </visual>
+          <mesh filename="package://jackal_kinova_gazebo/meshes/jackal-fender.stl" />
+        </geometry>
+        <material name="yellow" />
+      </visual>
+      <collision name="front_fender_collision">
+        <geometry>
+          <mesh filename="package://jackal_kinova_gazebo/meshes/jackal-fender.stl"
+            scale="1.2 1.2 1.0" />
+        </geometry>
+      </collision>
     </link>
   </xacro:unless>
@@ -156,10 +176,16 @@
       <visual>
         <geometry>
-          <mesh filename="package://jackal_kinova_gazebo/meshes/accessory_fender.stl"/>
-        </geometry>
-        <material name="yellow" />
-      </visual>
-    </link>
-    <link name="rear_fender_accessory_link"/>
+          <mesh filename="package://jackal_kinova_gazebo/meshes/accessory_fender.stl" />
+        </geometry>
+        <material name="yellow" />
+      </visual>
+      <collision name="rear_fender_collision">
+        <geometry>
+          <mesh filename="package://jackal_kinova_gazebo/meshes/jackal-fender.stl"
+            scale="1.2 1.2 1.0" />
+        </geometry>
+      </collision>
+    </link>
+    <link name="rear_fender_accessory_link" />
     <joint name="rear_fender_accessory_joint" type="fixed">
       <origin xyz="0.25629 0 0.07455" rpy="${PI} 0 0" />
@@ -169,5 +195,5 @@
   </xacro:if>
   <joint name="rear_fender_joint" type="fixed">
-    <origin xyz="0 0 0" rpy="0 0 ${PI}"/>
+    <origin xyz="0 0 0" rpy="0 0 ${PI}" />
     <parent link="chassis_link" />
     <child link="rear_fender_link" />
@@ -176,7 +202,8 @@
   <link name="imu_link">
     <inertial>
-      <mass value="0.001"/>
-      <origin xyz="0 0 0" rpy="0 0 0"/>
-      <inertia ixx="${dummy_inertia}" ixy="0.0" ixz="0.0" iyy="${dummy_inertia}" iyz="0.0" izz="${dummy_inertia}"/>
+      <mass value="0.001" />
+      <origin xyz="0 0 0" rpy="0 0 0" />
+      <inertia ixx="${dummy_inertia}" ixy="0.0" ixz="0.0" iyy="${dummy_inertia}" iyz="0.0"
+        izz="${dummy_inertia}" />
     </inertial>
   </link>
