Commit message: Fix collision sensor

File: jackal_kinova_gazebo/urdf/jackal.urdf.xacro (robot description, xacro)
@@ -127,4 +127,10 @@
         <material name="yellow" />
       </visual>
+      <collision name="front_fender_collision">
+        <geometry>
+          <mesh filename="package://jackal_kinova_gazebo/meshes/jackal-fender.stl"
+            scale="1.2 1.2 1.0" />
+        </geometry>
+      </collision>
     </link>
   </xacro:unless>
@@ -164,5 +170,5 @@
         <material name="yellow" />
       </visual>
-      <collision name="front_fender_collision">
+      <collision name="rear_fender_collision">
         <geometry>
           <mesh filename="package://jackal_kinova_gazebo/meshes/jackal-fender.stl"
